File: design/Rosco I2C.kicad_sch (KiCad schematic)
At the start: 22 parts, among them J1 I2C Connector, J2 Rosco M68k Connector, J3 I2C Connector, J4 SPI, J5 Future, U2 74HC245, U3 GAL16V8, U4 GAL16V8, Y1 Crystal

Commit message: Checkpoint.  Working with AVR
Parts:
- removed C1, C6: 15pf, Capacitor_THT:C_Rect_L4.0mm_W2.5mm_P2.50mm, symbol Device:C
- removed C9: .1uF, Capacitor_THT:C_Rect_L4.0mm_W2.5mm_P2.50mm, symbol Device:C
- removed J3: I2C Connector, Connector_PinHeader_2.54mm:PinHeader_1x04_P2.54mm_Vertical, symbol Connector:Conn_01x04_Female
- removed J5: Future, Connector_PinSocket_2.54mm:PinSocket_1x08_P2.54mm_Vertical, symbol Connector:Conn_01x08_Female
- removed U?: ATmega32A-P, Package_DIP:DIP-40_W15.24mm, symbol MCU_Microchip_ATmega:ATmega32A-P
- removed Y1: Crystal, Crystal:Crystal_HC49-4H_Vertical, symbol Device:Crystal
- added C?: .1uF, Capacitor_SMD:C_0603_1608Metric, symbol Device:C
- added C?: .1uF, Capacitor_THT:C_Rect_L4.0mm_W2.5mm_P2.50mm, symbol Device:C
- added R? (x3): 10k, symbol Device:R
- added U?: ATmega1284-P, Package_DIP:DIP-40_W15.24mm, symbol MCU_Microchip_ATmega:ATmega1284-P
- added U?: 74HC245, Package_DIP:DIP-20_W7.62mm_Socket_LongPads, symbol 74xx:74HC245
- added X?: 16Mhz, Oscillator:Oscillator_DIP-8, symbol mc68k:CXO_DIP8
Connections:
- net A1: now also U?.2 (PB1)
- net A2: now also U?.3 (PB2)
- net A3: now also U?.4 (PB3)
- net A4: now also U?.5 (PB4)
- net A5: now also J4.3 (Pin_3), U?.6 (PB5)
- net A6: now also J4.6 (Pin_6), U?.7 (PB6)
- net A7: now also J4.4 (Pin_4), U?.8 (PB7)
- net CLK: now also U4.1 (I1/CLK), U?.13 (XTAL1), X?.5 (OUT)
- net D0: now also U?.2 (A0), U?.40 (PA0)
- net D1: now also U?.3 (A1), U?.39 (PA1)
- net D2: now also U?.38 (PA2), U?.4 (A2)
- net D3: now also U?.37 (PA3), U?.5 (A3)
- net D4: now also U?.36 (PA4), U?.6 (A4)
- net D5: now also U?.35 (PA5), U?.7 (A5); no longer J4.3 (Pin_3)
- net D6: now also U?.34 (PA6), U?.8 (A6); no longer J4.6 (Pin_6)
- net D7: now also U?.33 (PA7), U?.9 (A7); no longer J4.4 (Pin_4)
- net FC0: no longer U4.5 (I5)
- net FC1: no longer U4.6 (I6)
- net FC2: no longer U4.7 (I7)
- net GND: now also C?.2, C?.2, R?.2, R?.2, U?.10 (GND), U?.11 (GND), U?.31 (GND), X?.4 (GND)
- net RX: now also U?.15 (PD1)
- net R~{W}: now also U4.3 (I3), U?.1 (A->B), U?.19 (PD5); no longer U4.2 (I2)
- net SCL: now also U?.22 (PC0)
- net SDA: now also U?.23 (PC1)
- net TX: now also U?.14 (PD0)
- net VCC: now also C?.1, C?.1, R?.1, U?.10 (VCC), U?.20 (VCC), U?.30 (AVCC), U?.32 (AREF), X?.8 (Vcc)
- net ~{AS}: now also U4.4 (I4), U?.16 (PD2); no longer U4.3 (I3)
- net ~{DTACK_I2C}: now also U?.21 (PD7)
- net ~{I2CENABLE}: now also U?.17 (PD3); no longer U2.19 (CE)
- net ~{I2CSEL}: now also U4.2 (I2); no longer U4.1 (I1/CLK)
- net ~{LDS}: now also U4.5 (I5), U?.20 (PD6); no longer U4.4 (I4)
- net ~{RESET}: now also U?.9 (~{RESET})
- net ~{UDS}: now also U4.6 (I6)
- net ~{VPA}: no longer U4.8 (I8)
- net ~{UDSENABLE}: now reaches U4.16 (IO4)
- net ~{UDSENABLE}: now also U2.19 (CE), R?.1
- net ~{LDSENABLE}: now reaches U4.17 (I03)
- net ~{LDSENABLE}: now also R?.1, U?.19 (CE)
- net D10 renamed BUSD10
- net BUSD10: now also U?.16 (B2)
- net D11 renamed BUSD11
- net BUSD11: now also U?.15 (B3)
- net D12 renamed BUSD12
- net BUSD12: now also U?.14 (B4)
- net D13 renamed BUSD13
- net BUSD13: now also U?.13 (B5)
- net D14 renamed BUSD14
- net BUSD14: now also U?.12 (B6)
- net D15 renamed BUSD15
- net BUSD15: now also U?.11 (B7)
- net D8 renamed BUSD8
- net BUSD8: now also U?.18 (B0)
- net D9 renamed BUSD9
- net BUSD9: now also U?.17 (B1)
- new net: R?.2, U?.1 (PB0)
- no-connect marks 8 -> 15
Other:
- note added: "/I2CENBL = /I2CSEL * /AS * /LDS /UDSENABLE = /I2CSEL * /AS * /UDS /LDSENABLE = /I2CSEL * /AS * /LDS DTACK.T = GND DTACK.E = /DTACKI2C"
- note added: "I2CENABLE triggers INT1 to process"
- note removed: "/I2CENBL = /I2CSEL * /AS * /LDS DTACK.T = GND DTACK.E = /I2CSEL * /DTACKI2C"
- moved on the sheet: C10, C11, C2, C3, C4, C5, C7, C8, J1, J4, J?, U2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
